File: Circuit/boneIO - relay board 24x16A/boneIO - relay board.kicad_pcb (KiCad board)
At the start: 2 copper layers, 197 x 102 mm, 68 parts, among them J1 Screw_Terminal_01x04, J10 Screw_Terminal_01x04, J11 Screw_Terminal_01x04, J12 Screw_Terminal_01x04, J13 Screw_Terminal_01x04, J2 Screw_Terminal_01x04, J3 Conn_02x04_Odd_Even, J4 Screw_Terminal_01x04, J5 Screw_Terminal_01x04, J6 Screw_Terminal_01x04, J7 Screw_Terminal_01x04, J8 Screw_Terminal_01x04, J9 Screw_Terminal_01x04, SW1 SW_DIP_x03, SW2 SW_DIP_x03, SW3 SW_DIP_x03, U1 MCP9808-E_MS, U10 RM85-2011-35-1024, U11 RM85-2011-35-1024, U12 RM85-2011-35-1024, U13 RM85-2011-35-1024, U14 RM85-2011-35-1024, U15 RM85-2011-35-1024, U16 RM85-2011-35-1024, U17 RM85-2011-35-1024, U18 RM85-2011-35-1024, U19 RM85-2011-35-1024, U2 MCP23017_SS, U20 RM85-2011-35-1024, U21 RM85-2011-35-1024, U22 RM85-2011-35-1024, U23 RM85-2011-35-1024, U24 RM85-2011-35-1024, U25 RM85-2011-35-1024, U26 RM85-2011-35-1024, U27 RM85-2011-35-1024, U28 RM85-2011-35-1024, U29 RM85-2011-35-1024, U3 MCP23017_SS, U30 RM85-2011-35-1024, U4 ULN2803A, U5 ULN2803A, U6 ULN2803A, U7 RM85-2011-35-1024, U8 RM85-2011-35-1024, U9 RM85-2011-35-1024

Commit message: 24x16 v0.3
Parts:
- removed the R12 at (399.2, 317.9)
- removed the R8 at (354.2, 313.7)
- removed SW1, SW2, SW3: SW_DIP_x03, Button_Switch_SMD:SW_DIP_SPSTx03_Slide_KingTek_DSHP03TJ_W5.25mm_P1.27mm_JPin
- added JP1: NO_Small, Jumper:SolderJumper-2_P1.3mm_Open_RoundedPad1.0x1.5mm, F.Cu at (463.4, 308.8)
- added JP10: NO_Small, Jumper:SolderJumper-2_P1.3mm_Open_RoundedPad1.0x1.5mm, F.Cu at (399.2, 311.7)
- added JP2: NO_Small, Jumper:SolderJumper-2_P1.3mm_Open_RoundedPad1.0x1.5mm, F.Cu at (463.4, 310.9)
- added JP3: NO_Small, Jumper:SolderJumper-2_P1.3mm_Open_RoundedPad1.0x1.5mm, F.Cu at (463.4, 313.1)
- added JP5: NO_Small, Jumper:SolderJumper-2_P1.3mm_Open_RoundedPad1.0x1.5mm, F.Cu at (353.6, 318.6)
- added JP6: NO_Small, Jumper:SolderJumper-2_P1.3mm_Open_RoundedPad1.0x1.5mm, F.Cu at (351.0, 318.6)
- added JP7: NO_Small, Jumper:SolderJumper-2_P1.3mm_Open_RoundedPad1.0x1.5mm, F.Cu at (348.4, 318.6)
- added JP8: NO_Small, Jumper:SolderJumper-2_P1.3mm_Open_RoundedPad1.0x1.5mm, F.Cu at (404.0, 311.7)
- added JP9: NO_Small, Jumper:SolderJumper-2_P1.3mm_Open_RoundedPad1.0x1.5mm, F.Cu at (401.6, 311.7)
- added R14: 10k, Resistor_SMD:R_0603_1608Metric, F.Cu at (401.6, 316.5)
- added R15: 10k, Resistor_SMD:R_0603_1608Metric, F.Cu at (399.2, 316.5)
- added R2: 10k, Resistor_SMD:R_0603_1608Metric, F.Cu at (456.2, 311.0)
- added U1: MCP9808-E_SO8, Package_SO:SO-8_3.9x4.9mm_P1.27mm, F.Cu at (458.4, 317.8)
- R4: value 10k -> 4.7k
- moved R11 53.7 mm to (348.4, 313.8), turned to 90 degrees
- moved R5 12.1 mm to (464.5, 318.0), turned to 270 degrees
- moved R4 11.4 mm to (465.3, 315.6), turned to 0 degrees
- moved C1 10.4 mm to (466.3, 318.0), turned to 270 degrees
- moved R13 7.76 mm to (404.0, 316.5)
- moved R8 7.35 mm to (345.8, 318.5), turned to 90 degrees
- moved R10 4.57 mm to (351.0, 313.8), turned to 90 degrees
- moved R1 3.51 mm to (456.2, 309.3), turned to 180 degrees
- moved C3 3.22 mm to (357.4, 318.5), turned to 90 degrees
- moved R12 2.28 mm to (406.5, 316.5)
- moved U2 2.00 mm to (458.4, 317.8), turned to 270 degrees
- moved R9 1.65 mm to (353.6, 313.8), turned to 90 degrees
- moved R3 0.35 mm to (456.2, 312.7), turned to 180 degrees
- renumbered C4 to C2, C5 to C3, C6 to C4, C2 to C5, C3 to C6, JP1 to JP4, U7 to K1, U16 to K10, U17 to K11, U18 to K12, U19 to K13, U20 to K14, U21 to K15, U22 to K16, U23 to K17, U24 to K18, U25 to K19, U8 to K2, U26 to K20, U27 to K21, U28 to K22, U29 to K23, U30 to K24, U9 to K3, U10 to K4, U11 to K5, U12 to K6, U13 to K7, U14 to K8, U15 to K9, R14 to R12, R6 to R5, R5 to R6, R2 to R7, R7 to R8, U1 to U2, U4 to U3, U5 to U4, U6 to U5, U2 to U6, U3 to U7
Connections:
- R10 pad 1: Net-(R10-Pad1) -> Net-(JP6-Pad2)
- R11 pad 1: Net-(R11-Pad1) -> Net-(JP7-Pad2)
- R13 pad 1: Net-(R13-Pad1) -> Net-(JP8-Pad2)
- R3 pad 1: Net-(R3-Pad1) -> Net-(JP3-Pad2)
- R4 pad 1: Net-(R4-Pad1) -> +3V3
- R4 pad 2: GND -> Net-(R4-Pad2)
- R9 pad 1: Net-(R9-Pad1) -> Net-(JP5-Pad2)
- U2 pad 5: Net-(R4-Pad1) -> Net-(JP3-Pad2)
- U2 pad 6: Net-(R3-Pad1) -> Net-(JP2-Pad2)
- U6 pad 15: Net-(R10-Pad1) -> Net-(JP7-Pad2)
- U6 pad 16: Net-(R9-Pad1) -> Net-(JP6-Pad2)
- U6 pad 17: Net-(R8-Pad1) -> Net-(JP5-Pad2)
- U7 pad 15: Net-(R13-Pad1) -> Net-(JP10-Pad2)
- U7 pad 17: Net-(R11-Pad1) -> Net-(JP8-Pad2)
Routing:
- net Net-(JP10-Pad2): track 0.00 -> 27.2 mm, vias 0 -> 2
- net Net-(R4-Pad2): track 0.00 -> 22.4 mm, vias 0 -> 2
- net Net-(JP2-Pad2): track 0.00 -> 22.0 mm, vias 0 -> 3
- net Net-(JP3-Pad2): track 0.00 -> 20.8 mm, vias 0 -> 3
- net Net-(R10-Pad1): track 19.0 -> 0.00 mm
- net Net-(JP5-Pad2): track 0.00 -> 18.4 mm
- net Net-(R13-Pad1): track 17.8 -> 0.00 mm
- net Net-(R5-Pad2): track 3.66 -> 21.2 mm, vias 0 -> 2
- net Net-(R9-Pad1): track 16.5 -> 0.00 mm
- net Net-(JP9-Pad2): track 14.3 -> 30.3 mm, vias 0 -> 2
- net Net-(R8-Pad1): track 14.9 -> 0.00 mm
- net Net-(JP6-Pad2): track 0.00 -> 14.8 mm, vias 0 -> 2
- net Net-(R3-Pad1): track 12.6 -> 0.00 mm
- net Net-(JP7-Pad2): track 0.00 -> 12.2 mm
- net Net-(R4-Pad1): track 11.9 -> 0.00 mm
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Other:
- board text added: "Relay Board 24x16A v0.3"
- board text removed: "Relay Board 24x16A"

Commit message: update
Parts:
- A0: renamed from JP10; moved to B.Cu
- A0: renamed from JP7; moved to B.Cu
- A1: renamed from JP9; moved to B.Cu
- A1: renamed from JP6; moved to B.Cu
- A2: renamed from JP8; moved to B.Cu
- A2: renamed from JP5; moved to B.Cu
- JP1, JP2, JP3: moved to B.Cu
- moved A0 1.69 mm to (399.2, 310.1)
- moved A1 1.69 mm to (401.6, 310.0)
- moved A2 1.69 mm to (404.0, 310.0)
- moved A1 0.58 mm to (350.9, 319.2)
- moved A2 0.56 mm to (353.5, 319.2)
- moved A0 0.55 mm to (348.3, 319.2)
Routing:
- net +3V3: track 262.7 -> 235.4 mm, vias 9 -> 12
- net Net-(JP10-Pad2): track 27.2 -> 31.5 mm, vias 2 -> 3
- net SCL: track 141.4 -> 144.7 mm
- net Net-(JP8-Pad2): track 8.45 -> 10.2 mm, vias 0 -> 1
- net Net-(JP9-Pad2): track 30.3 -> 31.8 mm, vias 2 -> 3
- net Net-(JP6-Pad2): track 14.8 -> 15.6 mm
- net Net-(JP5-Pad2): track 18.4 -> 19.0 mm, vias 0 -> 1
- net Net-(JP7-Pad2): track 12.2 -> 12.6 mm, vias 0 -> 1
- net Net-(JP3-Pad2): vias 3 -> 4
- net Net-(JP2-Pad2): vias 3 -> 4
Other:
- board text added: "DOWN"
- board text added: "WARNING!!!"
