File: Circuit/boneIO - relay board 24x16A/boneIO - relay board.sch (KiCad schematic (older format))
At the start: 67 parts, among them J1 Screw_Terminal_01x04, J10 Screw_Terminal_01x04, J11 Screw_Terminal_01x04, J12 Screw_Terminal_01x04, J13 Screw_Terminal_01x04, J2 Screw_Terminal_01x04, J3 Conn_02x04_Odd_Even, J4 Screw_Terminal_01x04, J5 Screw_Terminal_01x04, J6 Screw_Terminal_01x04, J7 Screw_Terminal_01x04, J8 Screw_Terminal_01x04, J9 Screw_Terminal_01x04, K1 RM85-2011-35-1005, K10 RM85-2011-35-1005, K11 RM85-2011-35-1005, K12 RM85-2011-35-1005, K13 RM85-2011-35-1005, K14 RM85-2011-35-1005, K15 RM85-2011-35-1005, K16 RM85-2011-35-1005, K17 RM85-2011-35-1005, K18 RM85-2011-35-1005, K19 RM85-2011-35-1005, K2 RM85-2011-35-1005, K20 RM85-2011-35-1005, K21 RM85-2011-35-1005, K22 RM85-2011-35-1005, K23 RM85-2011-35-1005, K24 RM85-2011-35-1005, K3 RM85-2011-35-1005, K4 RM85-2011-35-1005, K5 RM85-2011-35-1005, K6 RM85-2011-35-1005, K7 RM85-2011-35-1005, K8 RM85-2011-35-1005, K9 RM85-2011-35-1005, SW1 SW_DIP_x03, SW2 SW_DIP_x03, SW3 SW_DIP_x03, U1 MCP9808_MSOP, U2 MCP23017_SS, U3 MCP23017_SS, U4 ULN2803A, U5 ULN2803A, U6 ULN2803A

Commit message: DRC Cleanup and some other small fixes
Parts:
- J3: footprint Connector_PinSocket_2.54mm:PinSocket_2x04_P2.54mm_Vertical -> ph80ds-21:PinHeader_2x04_P2.54mm_Vertical
Changed lines of the file:
@@
 F 0 "J3" H 6400 3667 50  0000 C CNN
 F 1 "Conn_02x04_Odd_Even" H 6400 3576 50  0000 C CNN
-F 2 "Connector_PinSocket_2.54mm:PinSocket_2x04_P2.54mm_Vertical" H 6350 3350 50  0001 C CNN
+F 2 "ph80ds-21:PinHeader_2x04_P2.54mm_Vertical" H 6350 3350 50  0001 C CNN
 F 3 "~" H 6350 3350 50  0001 C CNN
 	1    6350 3350

Commit message: cleanup relay board 24x16
Parts:
- J3: footprint ph80ds-21:PinHeader_2x04_P2.54mm_Vertical -> boneIO:PinHeader_2x04_P2.54mm_Vertical
- K1, K10, K11, K12, K13, K14, K15, K16, K17, K18, K19, K2, K20, K21, K22, K23, K24, K3, K4, K5, K6, K7, K8, K9: footprint boneIO - RM85:RM852011351005_1 -> boneIO:RM852011351005_1; symbol boneIO---relay-board-rescue:RM85-2011-35-1005-MK-boneIO---relay-board-rescue -> boneIO:RM85-2011-35-1005
- U1: symbol boneIO---relay-board-rescue:MCP9808_MSOP-Sensor_Temperature-boneIO---relay-board-rescue -> boneIO:MCP9808_MSOP

Commit message: 24x16 cleanup
Parts:
- removed K1, K10, K11, K12, K13, K14, K15, K16, K17, K18, K19, K2, K20, K21, K22, K23, K24, K3, K4, K5, K6, K7, K8, K9: RM85-2011-35-1005, boneIO:RM852011351005_1, symbol boneIO:RM85-2011-35-1005
- removed U1: MCP9808_MSOP, Package_SO:MSOP-8_3x3mm_P0.65mm, symbol boneIO:MCP9808_MSOP
- added U1: MCP9808-E_MS, boneIO - relay board 24x16A:SOP65P490X110-8N, symbol boneIO:MCP9808-E_MS
- added U10, U11, U12, U13, U14, U15, U16, U17, U18, U19, U20, U21, U22, U23, U24, U25, U26, U27, U28, U29, U30, U7, U8, U9: RM85-2011-35-1024, boneIO - relay board 24x16A:RM852011351024, symbol boneIO:RM85-2011-35-1024
- J3: footprint boneIO:PinHeader_2x04_P2.54mm_Vertical -> boneIO - relay board 24x16A:PinHeader_2x04_P2.54mm_Vertical
Connections:
- net +3V3: now also U1.8 (VDD)
- net GND: now also U1.4 (GND)
- net RELAY1: now also U7.A1
- net RELAY10: now also U16.A1
- net RELAY11: now also U17.A1
- net RELAY12: now also U18.A1
- net RELAY13: now also U22.A1
- net RELAY14: now also U21.A1
- net RELAY15: now also U20.A1
- net RELAY16: now also U19.A1
- net RELAY17: now also U23.A1
- net RELAY18: now also U24.A1
- net RELAY19: now also U25.A1
- net RELAY2: now also U8.A1
- net RELAY20: now also U26.A1
- net RELAY21: now also U27.A1
- net RELAY22: now also U28.A1
- net RELAY23: now also U29.A1
- net RELAY24: now also U30.A1
- net RELAY3: now also U9.A1
- net RELAY4: now also U10.A1
- net RELAY5: now also U11.A1
- net RELAY6: now also U12.A1
- net RELAY7: now also U13.A1
- net RELAY8: now also U14.A1
- net RELAY9: now also U15.A1
- net SCL: now also U1.2 (SCL)
- net SDA: now also U1.1 (SDA)
- net VCC: now also U10.A2, U11.A2, U12.A2, U13.A2, U14.A2, U15.A2, U16.A2, U17.A2, U18.A2, U19.A2, U20.A2, U21.A2, U22.A2, U23.A2, U24.A2, U25.A2, U26.A2, U27.A2, U28.A2, U29.A2, U30.A2, U7.A2, U8.A2, U9.A2
- net at J13.1 (Pin_1): now also U29.11, U29.21
- net at J13.2 (Pin_2): now also U29.14, U29.24
- net at J13.3 (Pin_3): now also U30.11, U30.21
- net at J13.4 (Pin_4): now also U30.14, U30.24
- net at J12.1 (Pin_1): now also U27.11, U27.21
- net at J12.2 (Pin_2): now also U27.14, U27.24
- net at J12.3 (Pin_3): now also U28.11, U28.21
- net at J12.4 (Pin_4): now also U28.14, U28.24
- net at R4.1, SW1.4: now also U1.5 (A2)
- net at R3.1, SW1.5: now also U1.6 (A1)
- net at R1.1, SW1.6: now also U1.7 (A0)
- net at R6.2: now also U1.3 (Alert)
- net at J1.1 (Pin_1): now also U7.11, U7.21
- net at J1.2 (Pin_2): now also U7.14, U7.24
- net at J1.3 (Pin_3): now also U8.11, U8.21
- net at J1.4 (Pin_4): now also U8.14, U8.24
- net at J2.3 (Pin_3): now also U10.11, U10.21
- net at J2.4 (Pin_4): now also U10.14, U10.24
- net at J2.1 (Pin_1): now also U9.11, U9.21
- net at J2.2 (Pin_2): now also U9.14, U9.24
- net at J4.3 (Pin_3): now also U12.11, U12.21
- net at J4.4 (Pin_4): now also U12.14, U12.24
- net at J4.1 (Pin_1): now also U11.11, U11.21
- net at J4.2 (Pin_2): now also U11.14, U11.24
- net at J5.3 (Pin_3): now also U14.11, U14.21
- net at J5.4 (Pin_4): now also U14.14, U14.24
- net at J5.1 (Pin_1): now also U13.11, U13.21
- net at J5.2 (Pin_2): now also U13.14, U13.24
- net at J6.3 (Pin_3): now also U16.11, U16.21
- net at J6.4 (Pin_4): now also U16.14, U16.24
- net at J6.1 (Pin_1): now also U15.11, U15.21
- net at J6.2 (Pin_2): now also U15.14, U15.24
- net at J7.1 (Pin_1): now also U18.11, U18.21
- net at J7.2 (Pin_2): now also U18.14, U18.24
- net at J7.3 (Pin_3): now also U17.11, U17.21
- net at J7.4 (Pin_4): now also U17.14, U17.24
- net at J9.1 (Pin_1): now also U21.11, U21.21
- net at J9.2 (Pin_2): now also U21.14, U21.24
- net at J9.3 (Pin_3): now also U22.11, U22.21
- net at J9.4 (Pin_4): now also U22.14, U22.24
- net at J8.1 (Pin_1): now also U19.11, U19.21
- net at J8.2 (Pin_2): now also U19.14, U19.24
- net at J8.3 (Pin_3): now also U20.11, U20.21
- net at J8.4 (Pin_4): now also U20.14, U20.24
- net at J10.1 (Pin_1): now also U24.11, U24.21
- net at J10.2 (Pin_2): now also U24.14, U24.24
- net at J10.3 (Pin_3): now also U23.11, U23.21
- net at J10.4 (Pin_4): now also U23.14, U23.24
- net at J11.1 (Pin_1): now also U26.11, U26.21
- net at J11.2 (Pin_2): now also U26.14, U26.24
- net at J11.3 (Pin_3): now also U25.11, U25.21
- net at J11.4 (Pin_4): now also U25.14, U25.24
- no-connect marks 60 -> 61
Other:
- moved on the sheet: C4, C5, C6, J1, J11, J2, J3, J4, J5, J6, J7, R1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

Commit message: 24x16 v0.3
Parts:
- removed R12, R8: 10k, Resistor_SMD:R_0603_1608Metric, symbol Device:R
- removed SW1, SW2, SW3: SW_DIP_x03, Button_Switch_SMD:SW_DIP_SPSTx03_Slide_KingTek_DSHP03TJ_W5.25mm_P1.27mm_JPin, symbol Switch:SW_DIP_x03
- added JP1, JP10, JP2, JP3, JP5, JP6, JP7, JP8, JP9: NO_Small, Jumper:SolderJumper-2_P1.3mm_Open_RoundedPad1.0x1.5mm, symbol Device:Jumper_NO_Small
- added R14, R15, R2: 10k, Resistor_SMD:R_0603_1608Metric, symbol Device:R
- added U1: MCP9808-E_SO8, Package_SO:SO-8_3.9x4.9mm_P1.27mm, symbol Sensor_Temperature:MCP9804_MSOP
- R4: value 10k -> 4.7k
- U2: renamed from U1; symbol boneIO:MCP9808-E_MS -> Sensor_Temperature:MCP9804_MSOP
- renumbered C4 to C2, C5 to C3, C6 to C4, C2 to C5, C3 to C6, JP1 to JP4, U7 to K1, U16 to K10, U17 to K11, U18 to K12, U19 to K13, U20 to K14, U21 to K15, U22 to K16, U23 to K17, U24 to K18, U25 to K19, U8 to K2, U26 to K20, U27 to K21, U28 to K22, U29 to K23, U30 to K24, U9 to K3, U10 to K4, U11 to K5, U12 to K6, U13 to K7, U14 to K8, U15 to K9, R14 to R12, R6 to R5, R5 to R6, R2 to R7, R7 to R8, U4 to U3, U5 to U4, U6 to U5, U2 to U6, U3 to U7
Connections:
- net +3V3: now also R4.1, JP1.1, JP10.1, JP2.1, JP3.1, JP5.1, JP6.1, JP7.1, JP8.1, JP9.1, U1.8 (VDD)
- net GND: now also R14.2, R15.2, R2.2, U1.4 (GND); no longer R4.2
- net SCL: now also U1.2 (SCL)
- net SDA: now also U1.1 (SDA)
- net at U2.5 (A2): now also R3.1, JP3.2, U1.5 (A2); no longer R4.1
- net at U2.6 (A1): now also JP2.2, R2.1, U1.6 (A1); no longer R3.1
- net at R1.1, U2.7 (A0): now also JP1.2, U1.7 (A0)
- net at U6.15 (A0): now also R11.1, JP7.2; no longer R10.1
- net at U6.16 (A1): now also R10.1, JP6.2; no longer R9.1
- net at U6.17 (A2): now also R9.1, JP5.2
- net at U7.15 (A0): now also JP10.2, R15.1; no longer R13.1
- net at U7.16 (A1): now also JP9.2, R14.1
- net at U7.17 (A2): now also R13.1, JP8.2; no longer R11.1
- new net: R4.2, U1.3 (Alert)
Other:
- note added: "- relay board 24x16A v0.3"
- note added: "ADDRESS\n 0x22\n"
- note added: "ADDRESS\n 0x23"
- note added: "ADDRESS\n 0x48"
- note removed: "boneIO - relay board 24x16A v0.2"
- moved on the sheet: C1, J1, J10, J11, J12, J13, J2, J4, J5, J6, J7, J8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
